File: trackerGPS/gpsModule.sch (KiCad schematic (older format))
At the start: 2 parts, among them IC5 L86-M33

Commit message: PCB completed with test points 	modified:   trackerGPS/gpsModule.bak 	modified:   trackerGPS/gpsModule.sch 	modified:   trackerGPS/microcontroller.bak 	modified:   trackerGPS/microcontroller.sch 	modified:   trackerGPS/powerSupply.bak 	modified:   trackerGPS/powerSupply.sch 	modified:   trackerGPS/simModule.bak 	modified:   trackerGPS/simModule.sch 	modified:   trackerGPS/trackerGPS-cache.lib 	modified:   trackerGPS/trackerGPS.bak 	modified:   trackerGPS/trackerGPS.kicad_pcb 	modified:   trackerGPS/trackerGPS.kicad_pcb-bak 	modified:   trackerGPS/trackerGPS.sch
Connections:
- wire segments 23 -> 15
Changed lines of the file:
@@
 $Descr A4 11693 8268
 encoding utf-8
-Sheet 4 5
+Sheet 3 5
 Title ""
 Date ""
@@
 L power:GND #PWR0110
 U 1 1 605AAD20
-P 7025 4225
-F 0 "#PWR0110" H 7025 3975 50  0001 C CNN
-F 1 "GND" H 7030 4052 50  0000 C CNN
-F 2 "" H 7025 4225 50  0001 C CNN
-F 3 "" H 7025 4225 50  0001 C CNN
-	1    7025 4225
+P 6225 3000
+F 0 "#PWR0110" H 6225 2750 50  0001 C CNN
+F 1 "GND" H 6230 2827 50  0000 C CNN
+F 2 "" H 6225 3000 50  0001 C CNN
+F 3 "" H 6225 3000 50  0001 C CNN
+	1    6225 3000
 	1    0    0    -1
 $EndComp
 Wire Wire Line
-	6775 3650 7025 3650
+	5975 2800 6225 2800
 Wire Wire Line
-	7025 3650 7025 3750
+	6225 2800 6225 2900
 Wire Wire Line
-	6775 3750 7025 3750
-Connection ~ 7025 3750
-Wire Wire Line
-	7025 3750 7025 3850
-Wire Wire Line
-	6775 3850 7025 3850
-Connection ~ 7025 3850
-Wire Wire Line
-	7025 3850 7025 3950
-Wire Wire Line
-	6775 3950 7025 3950
-Connection ~ 7025 3950
-Wire Wire Line
-	7025 3950 7025 4050
-Wire Wire Line
-	6775 4050 7025 4050
-Connection ~ 7025 4050
-Wire Wire Line
-	7025 4050 7025 4150
-Wire Wire Line
-	6775 4150 7025 4150
-Connection ~ 7025 4150
-Wire Wire Line
-	7025 4150 7025 4225
+	5975 2900 6225 2900
 Wire Wire Line
 	4375 2650 4575 2650
@@
 	4450 2550 4450 2450
 Connection ~ 4450 2450
+Wire Wire Line
+	6225 2900 6225 3000
+Connection ~ 6225 2900
 $EndSCHEMATC
