File: trackerGPS/powerSupply.sch (KiCad schematic (older format))
At the start: 6 parts, among them IC4 MAX17263LETD+, U1 REG113NA-3.3_3K, U2 1043P

Commit message: modified:   trackerGPS/microcontroller.bak 	modified:   trackerGPS/powerSupply.bak 	modified:   trackerGPS/powerSupply.sch 	modified:   trackerGPS/trackerGPS-cache.lib 	modified:   trackerGPS/trackerGPS.bak 	modified:   trackerGPS/trackerGPS.kicad_pcb 	modified:   trackerGPS/trackerGPS.kicad_pcb-bak
Parts:
- removed IC4: MAX17263LETD+, MAX17263LETD+:SON40P300X300X80-15N, symbol MAX17263LETD+:MAX17263LETD+
- added IC2: BQ24072TRGTT, Package_DFN_QFN:QFN-16-1EP_3x3mm_P0.5mm_EP2.7x2.7mm_ThermalVias, symbol BQ24072TRGTT:BQ24072TRGTT
- added J4: USB_A, USB_JAE:DX4R005HJ5, symbol Connector:USB_A
Changed lines of the file:
@@
 	3075 3325 3700 3325
 $Comp
-L MAX17263LETD+:MAX17263LETD+ IC4
-U 1 1 60637B23
-P 6875 2125
-F 0 "IC4" H 7575 2603 50  0000 C CNN
-F 1 "MAX17263LETD+" H 7575 2512 50  0000 C CNN
-F 2 "MAX17263LETD+:SON40P300X300X80-15N" H 8125 2225 50  0001 L CNN
-F 3 "https://datasheets.maximintegrated.com/en/ds/MAX17263.pdf" H 8125 2125 50  0001 L CNN
-F 4 "MAXIM INTEGRATED PRODUCTS - MAX17263LETD+ - SINGLE/MULTI-CELL FUEL GAUGE" H 8125 2025 50  0001 L CNN "Description"
-F 5 "0.8" H 8125 1925 50  0001 L CNN "Height"
-F 6 "Maxim Integrated" H 8125 1825 50  0001 L CNN "Manufacturer_Name"
-F 7 "MAX17263LETD+" H 8125 1725 50  0001 L CNN "Manufacturer_Part_Number"
-F 8 "700-MAX17263LETD+" H 8125 1625 50  0001 L CNN "Mouser Part Number"
-F 9 "https://www.mouser.com/Search/Refine.aspx?Keyword=700-MAX17263LETD%2B" H 8125 1525 50  0001 L CNN "Mouser Price/Stock"
-	1    6875 2125
+L Connector:USB_A J4
+U 1 1 6064EA36
+P 1550 4700
+F 0 "J4" H 1605 5167 50  0000 C CNN
+F 1 "USB_A" H 1605 5076 50  0000 C CNN
+F 2 "USB_JAE:DX4R005HJ5" H 1700 4650 50  0001 C CNN
+F 3 " ~" H 1700 4650 50  0001 C CNN
+	1    1550 4700
 	1    0    0    -1
 $EndComp
+$Comp
+L BQ24072TRGTT:BQ24072TRGTT IC2
+U 1 1 6064F3DC
+P 6275 1725
+F 0 "IC2" H 7516 1571 50  0000 L CNN
+F 1 "BQ24072TRGTT" H 7516 1480 50  0000 L CNN
+F 2 "Package_DFN_QFN:QFN-16-1EP_3x3mm_P0.5mm_EP2.7x2.7mm_ThermalVias" H 7325 2125 50  0001 L CNN
+F 3 "http://www.ti.com/lit/gpn/BQ24072T" H 7325 2025 50  0001 L CNN
+F 4 "1.5A USB-Friendly Li-Ion Battery Charger and Power-Path Management IC" H 7325 1925 50  0001 L CNN "Description"
+F 5 "1" H 7325 1825 50  0001 L CNN "Height"
+F 6 "Texas Instruments" H 7325 1725 50  0001 L CNN "Manufacturer_Name"
+F 7 "BQ24072TRGTT" H 7325 1625 50  0001 L CNN "Manufacturer_Part_Number"
+F 8 "595-BQ24072TRGTT" H 7325 1525 50  0001 L CNN "Mouser Part Number"
+F 9 "https://www.mouser.co.uk/ProductDetail/Texas-Instruments/BQ24072TRGTT/?qs=C44r%252BX3hXgJEm3wVYARorw%3D%3D" H 7325 1425 50  0001 L CNN "Mouser Price/Stock"
+F 10 "BQ24072TRGTT" H 7325 1325 50  0001 L CNN "Arrow Part Number"
+F 11 "https://www.arrow.com/en/products/bq24072trgtt/texas-instruments" H 7325 1225 50  0001 L CNN "Arrow Price/Stock"
+	1    6275 1725
+	1    0    0    -1
+$EndComp

Commit message: added battery charger BQ24072T 	modified:   trackerGPS/powerSupply.bak 	modified:   trackerGPS/powerSupply.sch 	modified:   trackerGPS/sym-lib-table 	modified:   trackerGPS/trackerGPS-cache.lib 	new file:   trackerGPS/trackerGPS-rescue.dcm 	new file:   trackerGPS/trackerGPS-rescue.lib 	modified:   trackerGPS/trackerGPS.kicad_pcb 	modified:   trackerGPS/trackerGPS.kicad_pcb-bak
Parts:
- removed C7: C_Small, Capacitor_SMD:C_0805_2012Metric_Pad1.15x1.40mm_HandSolder, symbol Device:C_Small
- removed U2: 1043P, 1043P:1043P, symbol 1043P:1043P
- added C? (x2): 4.7uF, Capacitor_SMD:C_0805_2012Metric_Pad1.15x1.40mm_HandSolder, symbol Device:C_Small
- added C?: 1uF, Capacitor_SMD:C_0805_2012Metric_Pad1.15x1.40mm_HandSolder, symbol Device:C_Small
- added D? (x2): LED_Small, LED_SMD:LED_0805_2012Metric, symbol Device:LED_Small
- added R? (x2): 1.5kOhm, Resistor_SMD:R_0805_2012Metric_Pad1.15x1.40mm_HandSolder, symbol Device:R_Small
- added R?: 49.9kOhm, Resistor_SMD:R_0805_2012Metric_Pad1.15x1.40mm_HandSolder, symbol Device:R_Small
- added R?: 200kOhm, Resistor_SMD:R_0805_2012Metric_Pad1.15x1.40mm_HandSolder, symbol Device:R_Small
- added R?: NP, Resistor_SMD:R_0805_2012Metric_Pad1.15x1.40mm_HandSolder, symbol Device:R_Small
- added R?: 0ohm, Resistor_SMD:R_0805_2012Metric_Pad1.15x1.40mm_HandSolder, symbol Device:R_Small
- added TP1: Battery_GND, TestPoint:TestPoint_Pad_2.0x2.0mm, symbol Connector:TestPoint
- added TP2: Battery+, TestPoint:TestPoint_Pad_2.0x2.0mm, symbol Connector:TestPoint
Connections:
- net labels added: USB_D+, USB_D-
- wire segments 20 -> 74
Other:
- note removed: "AJOUTER CHARGEUR BATTERIE"
- moved on the sheet: C8, C9, IC2, J4, U1

Commit message: Component placed 	modified:   trackerGPS/microcontroller.bak 	modified:   trackerGPS/microcontroller.sch 	modified:   trackerGPS/powerSupply.bak 	modified:   trackerGPS/powerSupply.sch 	modified:   trackerGPS/simModule.bak 	modified:   trackerGPS/simModule.sch 	modified:   trackerGPS/trackerGPS-cache.lib 	modified:   trackerGPS/trackerGPS.bak 	modified:   trackerGPS/trackerGPS.kicad_pcb 	modified:   trackerGPS/trackerGPS.kicad_pcb-bak 	modified:   trackerGPS/trackerGPS.sch
Parts:
- added C18: 470nF, Capacitor_SMD:C_0805_2012Metric_Pad1.15x1.40mm_HandSolder, symbol Device:C_Small
- added C21: 10uF, Capacitor_SMD:C_0805_2012Metric_Pad1.15x1.40mm_HandSolder, symbol Device:C_Small
- added R14: 900ohm, Resistor_SMD:R_0805_2012Metric_Pad1.15x1.40mm_HandSolder, symbol Device:R_Small
- added R17: 5.56kOhm, Resistor_SMD:R_0805_2012Metric_Pad1.15x1.40mm_HandSolder, symbol Device:R_Small
- added R18: 1kOhm, Resistor_SMD:R_0805_2012Metric_Pad1.15x1.40mm_HandSolder, symbol Device:R_Small
- added U2: TLV75201PDSQT, TLV75201PDSQT:SON40P200X200X80-11N, symbol TLV75201PDSQT:TLV75201PDSQT
- gave numbers to parts that had none: 11
Connections:
- net Vcc_3.8V is gone; now on net 3.8V_Bat_5V_USB: C8.1, U1.1 (VIN)
- net GND: now also C18.2, C21.2, R14.1, R18.1, U2.11 (EPAD), U2.2 (GND_1), U2.4 (GND_2)
- net VBUS: now reaches C7.1, IC2.13 (IN), J4.1 (VBUS), R10.2
- net 3.8V_Bat_5V_USB: now reaches C16.1, IC2.10 (OUT_1), IC2.11 (OUT_2), R12.2, R16.2
- net 3.8V_Bat_5V_USB: now also C21.1, U2.9 (IN1)
- net at IC2.16 (ISET): now also R14.2
- net USB_D+ renamed USB+
- net USB_D- renamed USB-
- new net: R17.1, R18.2, U2.1 (FB1)
- new net Vcc_3.5V: C18.1, R17.2, U2.10 (OUT1), U2.3 (EN1)
Other:
- note added: "VOUT = VFB × (1 + R1/ R2)\nVFB = 0.55V"
- moved on the sheet: C15, C16, C7, C8, C9, D1, D2, IC2, J4, R10, R11, R12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

Commit message: PCB completed with test points 	modified:   trackerGPS/gpsModule.bak 	modified:   trackerGPS/gpsModule.sch 	modified:   trackerGPS/microcontroller.bak 	modified:   trackerGPS/microcontroller.sch 	modified:   trackerGPS/powerSupply.bak 	modified:   trackerGPS/powerSupply.sch 	modified:   trackerGPS/simModule.bak 	modified:   trackerGPS/simModule.sch 	modified:   trackerGPS/trackerGPS-cache.lib 	modified:   trackerGPS/trackerGPS.bak 	modified:   trackerGPS/trackerGPS.kicad_pcb 	modified:   trackerGPS/trackerGPS.kicad_pcb-bak 	modified:   trackerGPS/trackerGPS.sch
Parts:
- removed J4: USB_A, USB_JAE:DX4R005HJ5, symbol Connector:USB_A
- added J4: USB_B_Micro, USB_JAE:DX4R005HJ5, symbol Connector:USB_B_Micro
- added TP4: TP_chg, TestPoint:TestPoint_Pad_D1.0mm, symbol Connector:TestPoint
- added TP5: TP_3v3_GPS, TestPoint:TestPoint_Pad_D1.0mm, symbol Connector:TestPoint
Connections:
- net GND: now also J4.5 (GND), J4.6 (Shield)
- net USB+: now also J4.3 (D+)
- net USB-: now also J4.2 (D-)
- net VBUS: now also J4.1 (VBUS)
- net Vcc_3.3V: now also TP5.1
- net 3.8V_Bat_5V_USB renamed 3.8V_Bat_OR_5V_USB
- net 3.8V_Bat_OR_5V_USB: now also TP4.1
Changed lines of the file:
@@
 $Descr A4 11693 8268
 encoding utf-8
-Sheet 5 5
+Sheet 4 5
 Title ""
 Date ""
@@
 $EndComp
 Wire Wire Line
-	8350 2600 8875 2600
+	8350 2600 8650 2600
 Wire Wire Line
 	8875 2725 8875 2600
@@
 Connection ~ 6700 2600
 $Comp
-L Connector:USB_A J4
-U 1 1 6064EA36
-P 1575 2750
-F 0 "J4" H 1630 3217 50  0000 C CNN
-F 1 "USB_A" H 1630 3126 50  0000 C CNN
-F 2 "USB_JAE:DX4R005HJ5" H 1725 2700 50  0001 C CNN
-F 3 " ~" H 1725 2700 50  0001 C CNN
-	1    1575 2750
-	1    0    0    -1
-$EndComp
-$Comp
-L BQ24072TRGTT:BQ24072TRGTT IC2
+L BQ24072TRGTT:BQ24072TRGTT IC?
 U 1 1 6064F3DC
 P 3175 2800
-AR Path="/6064F3DC" Ref="IC2"  Part="1"
+AR Path="/6064F3DC" Ref="IC?"  Part="1"
 AR Path="/6058CD04/6064F3DC" Ref="IC2"  Part="1"
 F 0 "IC2" H 4400 3525 50  0000 L CNN
@@
 	8250 950  8400 950
 Wire Wire Line
-	8400 950  9500 950
-Wire Wire Line
 	9500 950  9500 1025
 Connection ~ 8400 950
@@
 Connection ~ 6325 950
 Text Label 5325 2600 0    50   ~ 0
-3.8V_Bat_5V_USB
-Wire Wire Line
-	5750 2600 6700 2600
+3.8V_Bat_OR_5V_USB
+Wire Wire Line
+	5750 2600 6200 2600
 Wire Wire Line
 	6800 1900 6800 1800
 Connection ~ 6800 1800
+$Comp
+L Connector:USB_B_Micro J4
+U 1 1 6069F820
+P 1575 2750
+F 0 "J4" H 1630 3217 50  0000 C CNN
+F 1 "USB_B_Micro" H 1630 3126 50  0000 C CNN
+F 2 "USB_JAE:DX4R005HJ5" H 1725 2700 50  0001 C CNN
+F 3 "~" H 1725 2700 50  0001 C CNN
+	1    1575 2750
+	1    0    0    -1
+$EndComp
+$Comp
+L Connector:TestPoint TP4
+U 1 1 606CA98B
+P 6200 2325
+F 0 "TP4" H 6258 2445 50  0000 L CNN
+F 1 "TP_chg" H 6258 2354 50  0000 L CNN
+F 2 "TestPoint:TestPoint_Pad_D1.0mm" H 6400 2325 50  0001 C CNN
+F 3 "~" H 6400 2325 50  0001 C CNN
+	1    6200 2325
+	1    0    0    -1
+$EndComp
+Wire Wire Line
+	6200 2325 6200 2600
+Connection ~ 6200 2600
+Wire Wire Line
+	6200 2600 6700 2600
+$Comp
+L Connector:TestPoint TP5
+U 1 1 606CD78E
+P 8650 2500
+F 0 "TP5" H 8708 2620 50  0000 L CNN
+F 1 "TP_3v3_GPS" H 8708 2529 50  0000 L CNN
+F 2 "TestPoint:TestPoint_Pad_D1.0mm" H 8850 2500 50  0001 C CNN
+F 3 "~" H 8850 2500 50  0001 C CNN
+	1    8650 2500
+	1    0    0    -1
+$EndComp
+Wire Wire Line
+	8650 2500 8650 2600
+Connection ~ 8650 2600
+Wire Wire Line
+	8650 2600 8875 2600
+Wire Wire Line
+	8400 950  9500 950
 $EndSCHEMATC

Commit message: Replaced TLV75201 by REG113NA 	modified:   "Bilan energ\303\251tique tracker GPS.xlsx" 	modified:   trackerGPS/microcontroller.bak 	modified:   trackerGPS/powerSupply.bak 	modified:   trackerGPS/powerSupply.sch 	modified:   trackerGPS/trackerGPS-cache.lib 	modified:   trackerGPS/trackerGPS.bak 	modified:   trackerGPS/trackerGPS.kicad_pcb 	modified:   trackerGPS/trackerGPS.kicad_pcb-bak 	modified:   trackerGPS/trackerGPS.sch
Parts:
- removed C21: 10uF, Capacitor_SMD:C_0805_2012Metric_Pad1.15x1.40mm_HandSolder, symbol Device:C_Small
- removed R17: 5.56kOhm, Resistor_SMD:R_0805_2012Metric_Pad1.15x1.40mm_HandSolder, symbol Device:R_Small
- removed R18: 1kOhm, Resistor_SMD:R_0805_2012Metric_Pad1.15x1.40mm_HandSolder, symbol Device:R_Small
- removed U2: TLV75201PDSQT, TLV75201PDSQT:SON40P200X200X80-11N, symbol TLV75201PDSQT:TLV75201PDSQT
- added C19: 4.7uF, Capacitor_SMD:C_0805_2012Metric_Pad1.15x1.40mm_HandSolder, symbol Device:C_Small
- added R6: 0Ohm, Resistor_SMD:R_0805_2012Metric_Pad1.15x1.40mm_HandSolder, symbol Device:R_Small
- added TP8: GND, TestPoint:TestPoint_Pad_D1.0mm, symbol Connector:TestPoint
- added U2: REG113NA-3.3_3K, REG113NA:Texas_Instruments-DBV0005A-0-0-IPC_A, symbol REG113NA:REG113NA-3.3_3K
- C18: value 470nF -> 4.7uF
Connections:
- net Vcc_3.5V is gone; now on net Vcc_BAT_GSM: C18.1
- net GND: now also C19.2, TP8.1, U2.2 (GND)
- net Vcc_GPS_Enables: now also R6.1
- net 3.8V_Bat_OR_5V_USB renamed Vcc_BAT_GSM
- net Vcc_BAT_GSM: now also R6.2, U2.1 (VIN), U2.3 (Enable)
- net Vcc_3.3V renamed Vcc_3.3V_GPS
- new net Vcc_3.3V_UC: C19.1, U2.5 (VOUT)

Commit message: added BOM and first prototype ready
Parts:
- added D3: LED_Small, LED_SMD:LED_0805_2012Metric, symbol Device:LED_Small
- added R7: 1.9kOhm, Resistor_SMD:R_0805_2012Metric_Pad1.15x1.40mm_HandSolder, symbol Device:R_Small
- added S1: 450302014072, 450302014072:450302014072, symbol 450302014072:450302014072
- added TP9: TP_3v3_UC, TestPoint:TestPoint_Pad_D1.0mm, symbol Connector:TestPoint
- R14: value 900ohm -> 909 ohm
- R6: value 0Ohm -> 0ohm
Connections:
- net GND: now also D3.1 (K)
- net Vcc_3.3V_UC: now also TP9.1
- net Vcc_BAT_GSM: now also R7.2
- net at C15.1, IC2.2 (BAT_1), IC2.3 (BAT_2): now also S1.2 (NO); no longer TP2.1
- new net: S1.1 (COM), TP2.1
- new net: D3.2 (A), R7.1
Other:
- moved on the sheet: TP1, TP2, TP8
Changed lines of the file:
@@
 L power:GND #PWR0106
 U 1 1 60591B92
-P 5100 3850
-F 0 "#PWR0106" H 5100 3600 50  0001 C CNN
-F 1 "GND" H 5105 3677 50  0000 C CNN
-F 2 "" H 5100 3850 50  0001 C CNN
-F 3 "" H 5100 3850 50  0001 C CNN
-	1    5100 3850
+P 5450 5025
+F 0 "#PWR0106" H 5450 4775 50  0001 C CNN
+F 1 "GND" H 5455 4852 50  0000 C CNN
+F 2 "" H 5450 5025 50  0001 C CNN
+F 3 "" H 5450 5025 50  0001 C CNN
+	1    5450 5025
 	1    0    0    -1
 $EndComp
@@
 Wire Wire Line
 	6975 3075 6975 2800
-Wire Wire Line
-	6975 2800 7050 2800
 $Comp
 L Device:C_Small C8
@@
 Wire Wire Line
 	6700 2625 6700 2600
-Wire Wire Line
-	6700 2600 7050 2600
 Wire Wire Line
 	6700 2825 6700 2925
@@
 L Connector:TestPoint TP1
 U 1 1 60650D48
-P 5100 3700
-F 0 "TP1" H 5158 3820 50  0000 L CNN
-F 1 "Battery_GND" H 5158 3729 50  0000 L CNN
-F 2 "TestPoint:TestPoint_Pad_2.0x2.0mm" H 5300 3700 50  0001 C CNN
-F 3 "~" H 5300 3700 50  0001 C CNN
-	1    5100 3700
-	1    0    0    -1
-$EndComp
-Wire Wire Line
-	5100 3700 5100 3850
+P 5450 4875
+F 0 "TP1" H 5508 4995 50  0000 L CNN
+F 1 "Battery_GND" H 5508 4904 50  0000 L CNN
+F 2 "TestPoint:TestPoint_Pad_2.0x2.0mm" H 5650 4875 50  0001 C CNN
+F 3 "~" H 5650 4875 50  0001 C CNN
+	1    5450 4875
+	1    0    0    -1
+$EndComp
+Wire Wire Line
+	5450 4875 5450 5025
 $Comp
 L Connector:TestPoint TP2
 U 1 1 60651B8E
-P 4625 2975
-F 0 "TP2" H 4683 3095 50  0000 L CNN
-F 1 "Battery+" H 4683 3004 50  0000 L CNN
-F 2 "TestPoint:TestPoint_Pad_2.0x2.0mm" H 4825 2975 50  0001 C CNN
-F 3 "~" H 4825 2975 50  0001 C CNN
-	1    4625 2975
+P 5375 3250
+F 0 "TP2" H 5433 3370 50  0000 L CNN
+F 1 "Battery+" H 5433 3279 50  0000 L CNN
+F 2 "TestPoint:TestPoint_Pad_2.0x2.0mm" H 5575 3250 50  0001 C CNN
+F 3 "~" H 5575 3250 50  0001 C CNN
+	1    5375 3250
 	1    0    0    -1
 $EndComp
@@
 Wire Wire Line
 	5000 2600 5000 2550
-Wire Wire Line
-	4625 2975 4625 3150
-Connection ~ 4625 3150
 $Comp
 L Device:C_Small C7
@@
 P 3825 3975
 F 0 "R14" H 3725 3950 50  0000 R CNN
-F 1 "900ohm" H 3725 4025 50  0000 R CNN
+F 1 "909 ohm" H 3725 4025 50  0000 R CNN
 F 2 "Resistor_SMD:R_0805_2012Metric_Pad1.15x1.40mm_HandSolder" H 3825 3975 50  0001 C CNN
 F 3 "~" H 3825 3975 50  0001 C CNN
@@
 3.8V_Bat_OR_5V_USB
 Wire Wire Line
-	5750 2600 6200 2600
+	5750 2600 6075 2600
 $Comp
 L Connector:USB_B_Micro J4
@@
 Vcc_3.3V_UC
 Wire Wire Line
-	8300 1125 8825 1125
+	8300 1125 8500 1125
 $Comp
 L power:GND #PWR0153
 U 1 1 606D2023
-P 5450 4600
-F 0 "#PWR0153" H 5450 4350 50  0001 C CNN
-F 1 "GND" H 5455 4427 50  0000 C CNN
-F 2 "" H 5450 4600 50  0001 C CNN
-F 3 "" H 5450 4600 50  0001 C CNN
-	1    5450 4600
+P 6050 4750
+F 0 "#PWR0153" H 6050 4500 50  0001 C CNN
+F 1 "GND" H 6055 4577 50  0000 C CNN
+F 2 "" H 6050 4750 50  0001 C CNN
+F 3 "" H 6050 4750 50  0001 C CNN
+	1    6050 4750
 	1    0    0    -1
 $EndComp
@@
 L Connector:TestPoint TP8
 U 1 1 606D20A9
-P 5450 4425
-F 0 "TP8" H 5508 4545 50  0000 L CNN
-F 1 "GND" H 5508 4454 50  0000 L CNN
-F 2 "TestPoint:TestPoint_Pad_D1.0mm" H 5650 4425 50  0001 C CNN
-F 3 "~" H 5650 4425 50  0001 C CNN
-	1    5450 4425
-	1    0    0    -1
-$EndComp
-Wire Wire Line
-	5450 4425 5450 4600
+P 6050 4575
+F 0 "TP8" H 6108 4695 50  0000 L CNN
+F 1 "GND" H 6108 4604 50  0000 L CNN
+F 2 "TestPoint:TestPoint_Pad_D1.0mm" H 6250 4575 50  0001 C CNN
+F 3 "~" H 6250 4575 50  0001 C CNN
+	1    6050 4575
+	1    0    0    -1
+$EndComp
+Wire Wire Line
+	6050 4575 6050 4750
 Wire Wire Line
 	5850 1750 5750 1750
@@
 P 7050 2700
 F 0 "R6" H 6991 2654 50  0000 R CNN
-F 1 "0Ohm" H 6991 2745 50  0000 R CNN
+F 1 "0ohm" H 6991 2745 50  0000 R CNN
 F 2 "Resistor_SMD:R_0805_2012Metric_Pad1.15x1.40mm_HandSolder" H 7050 2700 50  0001 C CNN
 F 3 "~" H 7050 2700 50  0001 C CNN
@@
 	-1   0    0    1
 $EndComp
+$Comp
+L Device:LED_Small D3
+U 1 1 606DD3B4
+P 6075 3350
+F 0 "D3" H 6075 3585 50  0000 C CNN
+F 1 "LED_Small" H 6075 3494 50  0000 C CNN
+F 2 "LED_SMD:LED_0805_2012Metric" V 6075 3350 50  0001 C CNN
+F 3 "~" V 6075 3350 50  0001 C CNN
+	1    6075 3350
+	0    -1   -1   0
+$EndComp
+Connection ~ 7050 2600
 Connection ~ 7050 2800
 Wire Wire Line
+	7050 2600 7250 2600
+Wire Wire Line
+	6700 2600 7050 2600
+Wire Wire Line
 	7050 2800 7250 2800
-Connection ~ 7050 2600
-Wire Wire Line
-	7050 2600 7250 2600
+Wire Wire Line
+	6975 2800 7050 2800
+$Comp
+L Device:R_Small R7
+U 1 1 606DFE75
+P 6075 2950
+F 0 "R7" H 6016 2904 50  0000 R CNN
+F 1 "1.9kOhm" H 6016 2995 50  0000 R CNN
+F 2 "Resistor_SMD:R_0805_2012Metric_Pad1.15x1.40mm_HandSolder" H 6075 2950 50  0001 C CNN
+F 3 "~" H 6075 2950 50  0001 C CNN
+	1    6075 2950
+	-1   0    0    1
+$EndComp
+Wire Wire Line
+	6075 2850 6075 2600
+Connection ~ 6075 2600
+Wire Wire Line
+	6075 2600 6200 2600
+Wire Wire Line
+	6075 3050 6075 3250
+$Comp
+L power:GND #PWR0154
+U 1 1 606E54AA
+P 6075 3550
+F 0 "#PWR0154" H 6075 3300 50  0001 C CNN
+F 1 "GND" H 6080 3377 50  0000 C CNN
+F 2 "" H 6075 3550 50  0001 C CNN
+F 3 "" H 6075 3550 50  0001 C CNN
+	1    6075 3550
+	1    0    0    -1
+$EndComp
+Wire Wire Line
+	6075 3450 6075 3550
+$Comp
+L Connector:TestPoint TP9
+U 1 1 606E9B98
+P 8500 1025
+F 0 "TP9" H 8558 1145 50  0000 L CNN
+F 1 "TP_3v3_UC" H 8558 1054 50  0000 L CNN
+F 2 "TestPoint:TestPoint_Pad_D1.0mm" H 8700 1025 50  0001 C CNN
+F 3 "~" H 8700 1025 50  0001 C CNN
+	1    8500 1025
+	1    0    0    -1
+$EndComp
+Wire Wire Line
+	8500 1025 8500 1125
+Connection ~ 8500 1125
+Wire Wire Line
+	8500 1125 8825 1125
+$Comp
+L 450302014072:450302014072 S1
+U 1 1 606EA603
+P 5250 3300
+F 0 "S1" V 6025 3200 50  0000 L CNN
+F 1 "450302014072" V 6150 2975 50  0000 L CNN
+F 2 "450302014072:450302014072" H 6000 3400 50  0001 L CNN
+F 3 "http://www.farnell.com/datasheets/1913864.pdf" H 6000 3300 50  0001 L CNN
+F 4 "Through Hole Slide Switch SPDT On-On 100 mA@ 42 V dc Slide" H 6000 3200 50  0001 L CNN "Description"
+F 5 "2.65" H 6000 3100 50  0001 L CNN "Height"
+F 6 "Wurth Elektronik" H 6000 3000 50  0001 L CNN "Manufacturer_Name"
+F 7 "450302014072" H 6000 2900 50  0001 L CNN "Manufacturer_Part_Number"
+F 8 "710-450302014072" H 6000 2800 50  0001 L CNN "Mouser Part Number"
+F 9 "https://www.mouser.com/Search/Refine.aspx?Keyword=710-450302014072" H 6000 2700 50  0001 L CNN "Mouser Price/Stock"
+F 10 "7856478" H 6000 2600 50  0001 L CNN "RS Part Number"
+F 11 "http://uk.rs-online.com/web/p/products/7856478" H 6000 2500 50  0001 L CNN "RS Price/Stock"
+	1    5250 3300
+	0    1    1    0
+$EndComp
+Wire Wire Line
+	5250 3300 5375 3300
+Wire Wire Line
+	5375 3300 5375 3250
+Wire Wire Line
+	5050 3300 5050 3150
+Wire Wire Line
+	4625 3150 5050 3150
+Connection ~ 4625 3150
 $EndSCHEMATC
