File: trackerGPS/simModule.sch (KiCad schematic (older format))
At the start: 16 parts, among them J3 902-9235, U3 MFF2_E_SIM, U5 M95

Commit message: Component placed 	modified:   trackerGPS/microcontroller.bak 	modified:   trackerGPS/microcontroller.sch 	modified:   trackerGPS/powerSupply.bak 	modified:   trackerGPS/powerSupply.sch 	modified:   trackerGPS/simModule.bak 	modified:   trackerGPS/simModule.sch 	modified:   trackerGPS/trackerGPS-cache.lib 	modified:   trackerGPS/trackerGPS.bak 	modified:   trackerGPS/trackerGPS.kicad_pcb 	modified:   trackerGPS/trackerGPS.kicad_pcb-bak 	modified:   trackerGPS/trackerGPS.sch
Parts:
- removed AE1: Antenna_Chip, symbol Device:Antenna_Chip
- added J5: Conn_Coaxial, Connector_Coaxial:U.FL_Hirose_U.FL-R-SMT-1_Vertical, symbol Connector:Conn_Coaxial
Connections:
- net GND: now also J5.2 (Ext)
- net at R2.2, R3.1: now also J5.1 (In)
Changed lines of the file:
@@
 $Descr A4 11693 8268
 encoding utf-8
-Sheet 3 5
+Sheet 2 5
 Title ""
 Date ""
@@
 	7975 4850 8050 4850
 $Comp
-L Device:Antenna_Chip AE1
-U 1 1 605D03FF
-P 10475 4625
-F 0 "AE1" H 10654 4753 50  0000 L CNN
-F 1 "Antenna_Chip" H 10654 4662 50  0000 L CNN
-F 2 "" H 10375 4800 50  0001 C CNN
-F 3 "~" H 10375 4800 50  0001 C CNN
-	1    10475 4625
-	1    0    0    -1
-$EndComp
-$Comp
 L Device:C_Small C28
 U 1 1 605D5087
@@
 Wire Wire Line
 	5025 3000 5175 3000
+$Comp
+L Connector:Conn_Coaxial J5
+U 1 1 6069FB20
+P 10750 4750
+F 0 "J5" H 10849 4726 50  0000 L CNN
+F 1 "Conn_Coaxial" H 10849 4635 50  0000 L CNN
+F 2 "Connector_Coaxial:U.FL_Hirose_U.FL-R-SMT-1_Vertical" H 10750 4750 50  0001 C CNN
+F 3 " ~" H 10750 4750 50  0001 C CNN
+	1    10750 4750
+	1    0    0    -1
+$EndComp
+Wire Wire Line
+	10225 4750 10550 4750
+Connection ~ 10225 4750
+$Comp
+L power:GND #PWR?
+U 1 1 6069DC5A
+P 10750 5050
+F 0 "#PWR?" H 10750 4800 50  0001 C CNN
+F 1 "GND" H 10755 4877 50  0000 C CNN
+F 2 "" H 10750 5050 50  0001 C CNN
+F 3 "" H 10750 5050 50  0001 C CNN
+	1    10750 5050
+	1    0    0    -1
+$EndComp
+Wire Wire Line
+	10750 4950 10750 5050
 $EndSCHEMATC

Commit message: PCB completed with test points 	modified:   trackerGPS/gpsModule.bak 	modified:   trackerGPS/gpsModule.sch 	modified:   trackerGPS/microcontroller.bak 	modified:   trackerGPS/microcontroller.sch 	modified:   trackerGPS/powerSupply.bak 	modified:   trackerGPS/powerSupply.sch 	modified:   trackerGPS/simModule.bak 	modified:   trackerGPS/simModule.sch 	modified:   trackerGPS/trackerGPS-cache.lib 	modified:   trackerGPS/trackerGPS.bak 	modified:   trackerGPS/trackerGPS.kicad_pcb 	modified:   trackerGPS/trackerGPS.kicad_pcb-bak 	modified:   trackerGPS/trackerGPS.sch
Parts:
- removed FB1: Ferrite, symbol Device:Ferrite_Bead_Small
Connections:
- net UART_GSM_CTS: now also U5.23 (CTS); no longer U5.24 (RTS)
- net UART_GSM_RTS: now also U5.24 (RTS); no longer U5.23 (CTS)
- net Vcc_GSM: now also U5.33 (VBAT), U5.34 (VBAT)
Changed lines of the file:
@@
 	1    0    0    -1
 $EndComp
-Text HLabel 5025 2650 0    50   Output ~ 0
+Text HLabel 5025 2550 0    50   Output ~ 0
 UART_GSM_CTS
-Text HLabel 5025 2550 0    50   Input ~ 0
+Text HLabel 5025 2650 0    50   Input ~ 0
 UART_GSM_RTS
 $Comp
@@
 	1    0    0    -1
 $EndComp
-$Comp
-L Device:Ferrite_Bead_Small FB1
-U 1 1 605DC0F8
-P 7550 2200
-F 0 "FB1" V 7787 2200 50  0000 C CNN
-F 1 "Ferrite" V 7696 2200 50  0000 C CNN
-F 2 "" V 7480 2200 50  0001 C CNN
-F 3 "~" H 7550 2200 50  0001 C CNN
-	1    7550 2200
-	0    -1   -1   0
-$EndComp
 Wire Wire Line
 	8450 2250 8450 2200
@@
 	5000 2250 5175 2250
 Wire Wire Line
-	5025 2550 5175 2550
-Wire Wire Line
-	5025 2650 5175 2650
-Wire Wire Line
 	5025 2750 5175 2750
 Wire Wire Line
@@
 $EndComp
 Wire Wire Line
-	7375 2200 7450 2200
-Wire Wire Line
-	7650 2200 7725 2200
-Wire Wire Line
 	7725 2250 7725 2200
 Connection ~ 7725 2200
@@
 	3450 3650 5175 3650
 Connection ~ 3450 3650
-Wire Wire Line
-	2200 4475 3575 4475
 Text HLabel 5025 3000 0    50   Input ~ 0
 Sleep_GSM
@@
 Connection ~ 10225 4750
 $Comp
-L power:GND #PWR?
+L power:GND #PWR0155
 U 1 1 6069DC5A
 P 10750 5050
-F 0 "#PWR?" H 10750 4800 50  0001 C CNN
+F 0 "#PWR0155" H 10750 4800 50  0001 C CNN
 F 1 "GND" H 10755 4877 50  0000 C CNN
 F 2 "" H 10750 5050 50  0001 C CNN
@@
 Wire Wire Line
 	10750 4950 10750 5050
+Wire Wire Line
+	5025 2550 5175 2550
+Wire Wire Line
+	5025 2650 5175 2650
+Wire Wire Line
+	7375 2200 7725 2200
+Wire Wire Line
+	2200 4475 3575 4475
 $EndSCHEMATC

Commit message: added BOM and first prototype ready
Parts:
- removed J3: 902-9235, 902-9235:9029235, symbol RF:902-9235
- added J1: MS-156HF, MS-156HF:MS156HF, symbol MS-156HF:MS-156HF
- R2: value R_Small -> 0ohm
Connections:
- net GND: now also J1.MP1, J1.MP2
- net at U5.39 (RF_ANT): now also J1.A1
- net at R1.2, R2.1: now also J1.C1
Other:
- moved on the sheet: J5, R1, R2, R3
Changed lines of the file:
@@
 	2100 3650 3450 3650
-$Comp
-L RF:902-9235 J3
-U 1 1 605C86E5
-P 7800 4750
-F 0 "J3" H 8725 5015 50  0000 C CNN
-F 1 "902-9235" H 8725 4924 50  0000 C CNN
-F 2 "902-9235:9029235" H 9450 5150 50  0001 L CNN
-F 3 "https://componentsearchengine.com/Datasheets/1/902-9235.pdf" H 9450 5050 50  0001 L CNN
-F 4 "RF Connectors / Coaxial Connectors MicroSwitch PCB Strt Jack Surf Mnt 50 ohm" H 9450 4950 50  0001 L CNN "Description"
-F 5 "1.05" H 9450 4850 50  0001 L CNN "Height"
-F 6 "Amphenol" H 9450 4750 50  0001 L CNN "Manufacturer_Name"
-F 7 "902-9235" H 9450 4650 50  0001 L CNN "Manufacturer_Part_Number"
-F 8 "902-9235" H 9450 4550 50  0001 L CNN "Arrow Part Number"
-F 9 "523-902-9235" H 9450 4350 50  0001 L CNN "Mouser Part Number"
-F 10 "https://www.mouser.co.uk/ProductDetail/Amphenol-RF/902-9235?qs=mAH9sUMRCtuATpVFdEB2WA%3D%3D" H 9450 4250 50  0001 L CNN "Mouser Price/Stock"
-	1    7800 4750
-	1    0    0    -1
-$EndComp
 $Comp
 L Device:R_Small R1
 U 1 1 605CA300
-P 9700 4950
-F 0 "R1" H 9641 4904 50  0000 R CNN
-F 1 "R_Small" H 9641 4995 50  0000 R CNN
-F 2 "Resistor_SMD:R_0805_2012Metric_Pad1.15x1.40mm_HandSolder" H 9700 4950 50  0001 C CNN
-F 3 "~" H 9700 4950 50  0001 C CNN
-	1    9700 4950
+P 9500 4650
+F 0 "R1" H 9441 4604 50  0000 R CNN
+F 1 "R_Small" H 9441 4695 50  0000 R CNN
+F 2 "Resistor_SMD:R_0805_2012Metric_Pad1.15x1.40mm_HandSolder" H 9500 4650 50  0001 C CNN
+F 3 "~" H 9500 4650 50  0001 C CNN
+	1    9500 4650
 	-1   0    0    1
 $EndComp
 Wire Wire Line
-	9700 4850 9700 4750
-Wire Wire Line
-	9700 4750 9875 4750
-Wire Wire Line
-	10075 4750 10225 4750
-Wire Wire Line
-	10225 4750 10225 4850
+	9500 4550 9500 4450
+Wire Wire Line
+	9500 4450 9675 4450
+Wire Wire Line
+	9875 4450 10025 4450
+Wire Wire Line
+	10025 4450 10025 4550
 $Comp
 L power:GND #PWR0129
 U 1 1 605CBAD7
-P 9700 5125
-F 0 "#PWR0129" H 9700 4875 50  0001 C CNN
-F 1 "GND" H 9705 4952 50  0000 C CNN
-F 2 "" H 9700 5125 50  0001 C CNN
-F 3 "" H 9700 5125 50  0001 C CNN
-	1    9700 5125
+P 9500 4825
+F 0 "#PWR0129" H 9500 4575 50  0001 C CNN
+F 1 "GND" H 9505 4652 50  0000 C CNN
+F 2 "" H 9500 4825 50  0001 C CNN
+F 3 "" H 9500 4825 50  0001 C CNN
+	1    9500 4825
 	1    0    0    -1
 $EndComp
@@
 L power:GND #PWR0130
 U 1 1 605CBAFF
-P 10225 5125
-F 0 "#PWR0130" H 10225 4875 50  0001 C CNN
-F 1 "GND" H 10230 4952 50  0000 C CNN
-F 2 "" H 10225 5125 50  0001 C CNN
-F 3 "" H 10225 5125 50  0001 C CNN
-	1    10225 5125
-	1    0    0    -1
-$EndComp
-Wire Wire Line
-	10225 5050 10225 5125
-Wire Wire Line
-	9700 5125 9700 5050
+P 10025 4825
+F 0 "#PWR0130" H 10025 4575 50  0001 C CNN
+F 1 "GND" H 10030 4652 50  0000 C CNN
+F 2 "" H 10025 4825 50  0001 C CNN
+F 3 "" H 10025 4825 50  0001 C CNN
+	1    10025 4825
+	1    0    0    -1
+$EndComp
+Wire Wire Line
+	10025 4750 10025 4825
+Wire Wire Line
+	9500 4825 9500 4750
 $Comp
 L Device:R_Small R2
 U 1 1 605CD39A
-P 9975 4750
-F 0 "R2" V 10171 4750 50  0000 C CNN
-F 1 "R_Small" V 10080 4750 50  0000 C CNN
-F 2 "Resistor_SMD:R_0805_2012Metric_Pad1.15x1.40mm_HandSolder" H 9975 4750 50  0001 C CNN
-F 3 "~" H 9975 4750 50  0001 C CNN
-	1    9975 4750
+P 9775 4450
+F 0 "R2" V 9971 4450 50  0000 C CNN
+F 1 "0ohm" V 9880 4450 50  0000 C CNN
+F 2 "Resistor_SMD:R_0805_2012Metric_Pad1.15x1.40mm_HandSolder" H 9775 4450 50  0001 C CNN
+F 3 "~" H 9775 4450 50  0001 C CNN
+	1    9775 4450
 	0    -1   -1   0
 $EndComp
@@
 L Device:R_Small R3
 U 1 1 605CD3EB
-P 10225 4950
-F 0 "R3" H 10284 4996 50  0000 L CNN
-F 1 "R_Small" H 10284 4905 50  0000 L CNN
-F 2 "Resistor_SMD:R_0805_2012Metric_Pad1.15x1.40mm_HandSolder" H 10225 4950 50  0001 C CNN
-F 3 "~" H 10225 4950 50  0001 C CNN
-	1    10225 4950
-	1    0    0    -1
-$EndComp
-Wire Wire Line
-	9400 4750 9700 4750
-Connection ~ 9700 4750
+P 10025 4650
+F 0 "R3" H 10084 4696 50  0000 L CNN
+F 1 "R_Small" H 10084 4605 50  0000 L CNN
+F 2 "Resistor_SMD:R_0805_2012Metric_Pad1.15x1.40mm_HandSolder" H 10025 4650 50  0001 C CNN
+F 3 "~" H 10025 4650 50  0001 C CNN
+	1    10025 4650
+	1    0    0    -1
+$EndComp
+Connection ~ 9500 4450
 $Comp
 L power:GND #PWR0131
 U 1 1 605D11C4
-P 7975 4925
-F 0 "#PWR0131" H 7975 4675 50  0001 C CNN
-F 1 "GND" H 7980 4752 50  0000 C CNN
-F 2 "" H 7975 4925 50  0001 C CNN
-F 3 "" H 7975 4925 50  0001 C CNN
-	1    7975 4925
+P 8350 5025
+F 0 "#PWR0131" H 8350 4775 50  0001 C CNN
+F 1 "GND" H 8355 4852 50  0000 C CNN
+F 2 "" H 8350 5025 50  0001 C CNN
+F 3 "" H 8350 5025 50  0001 C CNN
+	1    8350 5025
 	1    0    0    -1
 $EndComp
@@
 L power:GND #PWR0132
 U 1 1 605D1244
-P 9475 4925
-F 0 "#PWR0132" H 9475 4675 50  0001 C CNN
-F 1 "GND" H 9480 4752 50  0000 C CNN
-F 2 "" H 9475 4925 50  0001 C CNN
-F 3 "" H 9475 4925 50  0001 C CNN
-	1    9475 4925
-	1    0    0    -1
-$EndComp
-Wire Wire Line
-	9400 4850 9475 4850
-Wire Wire Line
-	9475 4850 9475 4925
-Wire Wire Line
-	7975 4925 7975 4850
-Wire Wire Line
-	7975 4850 8050 4850
+P 8750 5025
+F 0 "#PWR0132" H 8750 4775 50  0001 C CNN
+F 1 "GND" H 8755 4852 50  0000 C CNN
+F 2 "" H 8750 5025 50  0001 C CNN
+F 3 "" H 8750 5025 50  0001 C CNN
+	1    8750 5025
+	1    0    0    -1
+$EndComp
 $Comp
 L Device:C_Small C28
@@
 	7375 4450 8050 4450
 Wire Wire Line
-	8050 4450 8050 4750
-Wire Wire Line
 	2700 3450 5175 3450
 Connection ~ 2700 3450
@@
 L Connector:Conn_Coaxial J5
 U 1 1 6069FB20
-P 10750 4750
-F 0 "J5" H 10849 4726 50  0000 L CNN
-F 1 "Conn_Coaxial" H 10849 4635 50  0000 L CNN
-F 2 "Connector_Coaxial:U.FL_Hirose_U.FL-R-SMT-1_Vertical" H 10750 4750 50  0001 C CNN
-F 3 " ~" H 10750 4750 50  0001 C CNN
-	1    10750 4750
-	1    0    0    -1
-$EndComp
-Wire Wire Line
-	10225 4750 10550 4750
-Connection ~ 10225 4750
+P 10550 4450
+F 0 "J5" H 10649 4426 50  0000 L CNN
+F 1 "Conn_Coaxial" H 10649 4335 50  0000 L CNN
+F 2 "Connector_Coaxial:U.FL_Hirose_U.FL-R-SMT-1_Vertical" H 10550 4450 50  0001 C CNN
+F 3 " ~" H 10550 4450 50  0001 C CNN
+	1    10550 4450
+	1    0    0    -1
+$EndComp
+Wire Wire Line
+	10025 4450 10350 4450
+Connection ~ 10025 4450
 $Comp
 L power:GND #PWR0155
 U 1 1 6069DC5A
-P 10750 5050
-F 0 "#PWR0155" H 10750 4800 50  0001 C CNN
-F 1 "GND" H 10755 4877 50  0000 C CNN
-F 2 "" H 10750 5050 50  0001 C CNN
-F 3 "" H 10750 5050 50  0001 C CNN
-	1    10750 5050
-	1    0    0    -1
-$EndComp
-Wire Wire Line
-	10750 4950 10750 5050
+P 10550 4750
+F 0 "#PWR0155" H 10550 4500 50  0001 C CNN
+F 1 "GND" H 10555 4577 50  0000 C CNN
+F 2 "" H 10550 4750 50  0001 C CNN
+F 3 "" H 10550 4750 50  0001 C CNN
+	1    10550 4750
+	1    0    0    -1
+$EndComp
+Wire Wire Line
+	10550 4650 10550 4750
 Wire Wire Line
 	5025 2550 5175 2550
@@
 Wire Wire Line
 	2200 4475 3575 4475
+$Comp
+L MS-156HF:MS-156HF J1
+U 1 1 606EE21E
+P 8050 4450
+F 0 "J1" H 9050 4125 50  0000 L CNN
+F 1 "MS-156HF" H 8900 4025 50  0000 L CNN
+F 2 "MS-156HF:MS156HF" H 8900 4750 50  0001 L CNN
+F 3 "https://eu.mouser.com/datasheet/2/185/MS-156HF_CL0358-0238-4-00_2d-1619062.pdf" H 8900 4650 50  0001 L CNN
+F 4 "RF Connectors / Coaxial Connectors RCPT COAX MS-156HF SMT" H 8900 4550 50  0001 L CNN "Description"
+F 5 "1.75" H 8900 4450 50  0001 L CNN "Height"
+F 6 "Hirose" H 8900 4350 50  0001 L CNN "Manufacturer_Name"
+F 7 "MS-156HF" H 8900 4250 50  0001 L CNN "Manufacturer_Part_Number"
+F 8 "798-MS156HF" H 8900 4150 50  0001 L CNN "Mouser Part Number"
+F 9 "https://www.mouser.co.uk/ProductDetail/Hirose-Connector/MS-156HF?qs=p6VZ%252BklCkRROl41byNpEGw%3D%3D" H 8900 4050 50  0001 L CNN "Mouser Price/Stock"
+	1    8050 4450
+	1    0    0    -1
+$EndComp
+Wire Wire Line
+	8350 4950 8350 5025
+Wire Wire Line
+	8750 4950 8750 5025
+Wire Wire Line
+	9050 4450 9500 4450
 $EndSCHEMATC
