File: trackerGPS/trackerGPS.kicad_pcb (KiCad board)
At the start: 4 copper layers, 60.8 x 33.6 mm, 74 parts, among them IC1 PIC32MM0256GPM028-I_ML, IC2 BQ24072TRGTT, IC5 L86-M33, J2 Conn, J3 902-9235, J4 USB_B_Micro, J5 Conn_Coaxial, Q2 BC847BW,115, U1 REG113NA-3.3_3K, U2 REG113NA-3.3_3K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

Commit message: added BOM and first prototype ready
Parts:
- removed J3: 902-9235, 902-9235:9029235
- added D3: LED_Small, LED_SMD:LED_0805_2012Metric, F.Cu at (157.5, 74.9)
- added J1: MS-156HF, MS-156HF:MS156HF, F.Cu at (113.2, 85.6)
- added R7: 1.9kOhm, Resistor_SMD:R_0805_2012Metric_Pad1.15x1.40mm_HandSolder, F.Cu at (157.5, 71.1)
- added S1: 450302014072, 450302014072:450302014072, F.Cu at (158.5, 85.8)
- added TP9: TP_3v3_UC, TestPoint:TestPoint_Pad_D1.0mm, B.Cu at (105.6, 90.1)
- R14: value 900ohm -> 909 ohm
- R2: value R_Small -> 0ohm
- R6: value 0Ohm -> 0ohm
- moved TP2 3.49 mm to (151.5, 93.8)
- moved TP1 3.02 mm to (148.4, 93.8)
- moved R16 0.31 mm to (155.7, 85.5)
Connections:
- TP2 pad 1: Net-(C15-Pad1) -> Net-(S1-Pad1)
Routing:
- net /microcontroller/VBUS: track 75.5 -> 36.5 mm, vias 6 -> 5
- net Net-(S1-Pad1): track 0.00 -> 11.8 mm, vias 0 -> 1
- net GND: track 109.2 -> 117.8 mm, vias 67 -> 186
- net Net-(C15-Pad1): track 18.3 -> 24.7 mm, vias 0 -> 1
- net Net-(D3-Pad2): track 0.00 -> 1.80 mm
- net /powerSupply/Vcc_3.3V_UC: track 56.0 -> 57.3 mm
- net /powerSupply/Vcc_BAT_GSM: track 40.2 -> 41.4 mm, vias 8 -> 9
- net Net-(C24-Pad1): track 27.8 -> 28.7 mm
- net Net-(J1-PadA1): track 4.93 -> 4.12 mm
Other:
- board text added: "Epaisseur entre couche 1 et 2 = 0.2mm"
- board text removed: "METTRE STITCHING VIAS METTRE INTERRUPTEUR Mettre LED power Epaisseur entre couche 1 et 2 = 0.2mm"
